Commit message: commit final

File: cora_description/urdf/macros.xacro (robot description, xacro)
@@ -13,4 +13,5 @@
   <xacro:include filename="$(find wamv_gazebo)/urdf/components/wamv_p3d.xacro" />
   <xacro:include filename="$(find wamv_gazebo)/urdf/components/wamv_pinger.xacro" />
+    <xacro:include filename="$(find wamv_gazebo)/urdf/components/sonar_sensor.xacro" />
   <!-- Include dynamics macros -->
   <xacro:include filename="$(find cora_description)/urdf/cora_dynamics_plugin.xacro" />

File: wamv_description/urdf/wamv_base.urdf.xacro (robot description, xacro)
@@ -1,4 +1,6 @@
 <?xml version="1.0"?>
 <robot xmlns:xacro="http://ros.org/wiki/xacro" name="wam-v">
+ <xacro:arg name="namespace" default="wamv"/>
+  <xacro:property name="namespace" value="$(arg namespace)" scope="global" />
   <!-- Macro for creating the main collisions as simple shapes. -->
   <xacro:macro name="main_collisions" params="prefix reflect:=1">

File: wamv_gazebo/urdf/components/sonar_sensor(test).xacro (robot description, xacro)
@@ -1,64 +1,47 @@
 <?xml version="1.0"?>
 <robot xmlns:xacro="http://ros.org/wiki/xacro">
-  <xacro:macro name="sonar_sensor" params="name parent *origin ros_topic update_rate min_range max_range field_of_view ray_count">
-    <joint name="${name}_joint" type="fixed">
+  <!-- MTK3339 Constants -->
+  <xacro:property name="sonar_depth" value="0.01454" />
+  <xacro:property name="sonar_width" value="0.0457" />
+  <xacro:property name="sonar_height" value="0.0213" />
+  <xacro:property name="sonar_mass" value="0.020" />
+  <!-- MTK3339 constants -->
+  <!-- Inertias Macros
+  <xacro:include filename="$(find jetbot_description)/urdf/includes/gazebo/inertias.xacro" />
+ -->
+  <xacro:include filename="$(find wamv_gazebo)/urdf/components/sonar_sensor.xacro" />
+  <xacro:macro name="sensor_sonar" params="name x y z R:=0 P:=0 Y:=0 ros_topic update_rate min_range max_range field_of_view ray_count">
+  <!-- Sonar HCSR04 -->
+    <joint name="${prefix}_${name}_joint" type="fixed">
+      <parent link="${parent}"/>
+      <child link="${prefix}_${name}_link"/>
       <xacro:insert_block name="origin" />
-      <parent link="${parent}"/>
-      <child link="${name}_link"/>
     </joint>
-    <link name="${name}_link">
-      <inertial>
-        <mass value="0.001" />
-        <origin xyz="0 0 0" rpy="0 0 0" />
-        <inertia ixx="0.000000017" ixy="0" ixz="0" iyy="0.000000017" iyz="0" izz="0.000000017" />
-      </inertial>
+    <link name="${prefix}_${name}_link">
       <visual>
-        <origin xyz="0 0 0" rpy="0 0 0" />
+        <origin xyz="0 -${sonar_width/2} -${sonar_height/2}" rpy="${pi/2} 0 ${pi/2}"/>
         <geometry>
-          <!--<box size="0.01 0.01 0.01" /> -->
-          <mesh filename="package://hector_sensors_description/meshes/sonar_sensor/max_sonar_ez4.dae"/>
+          <mesh filename="package://prueba2/src/vrx_gazebo/models/sonar/hcsr04.stl" scale="0.001 0.001 0.001"/>
         </geometry>
+        <material name="purple"/>
       </visual>
       <collision>
-        <origin xyz="0 0 0" rpy="0 0 0" />
+        <origin xyz="0 0 ${sonar_depth/2}" rpy="0 0 0"/>
         <geometry>
-          <box size="0.01 0.01 0.01" />
+          <box size="${sonar_width} ${sonar_height} ${sonar_depth}"/>
         </geometry>
       </collision>
+      <xacro:cuboid_inertia mass="${sonar_mass}" x="${sonar_width}" y="${sonar_height}" z="${sonar_depth}" />
     </link>
-    <gazebo reference="${name}_link">
-      <sensor type="ray" name="${name}">
-        <always_on>true</always_on>
-        <update_rate>${update_rate}</update_rate>
-        <pose>0 0 0 0 0 0</pose>
-        <visualize>false</visualize>
-        <ray>
-          <scan>
-            <horizontal>
-              <samples>${ray_count}</samples>
-              <resolution>1</resolution>
-              <min_angle>-${field_of_view/2}</min_angle>
-              <max_angle> ${field_of_view/2}</max_angle>
-            </horizontal>
-            <vertical>
-              <samples>${ray_count}</samples>
-              <resolution>1</resolution>
-              <min_angle>-${field_of_view/2}</min_angle>
-              <max_angle> ${field_of_view/2}</max_angle>
-            </vertical>
-          </scan>
-          <range>
-            <min>${min_range}</min>
-            <max>${max_range}</max>
-            <resolution>0.01</resolution>
-          </range>
-        </ray>
-        <plugin name="gazebo_ros_${name}_controller" filename="libhector_gazebo_ros_sonar.so">
-          <gaussianNoise>0.005</gaussianNoise>
-          <topicName>${ros_topic}</topicName>
-          <frameId>${name}_link</frameId>
-        </plugin>
-      </sensor>
-    </gazebo>
+    <!-- Sonar Plugin -->
+    <xacro:gazebo_sonar name="${prefix}_${name}"
+                        reference_link="${prefix}_${name}_link"
+                        topic_ns="${name}"
+                        update_rate="10"
+                        min_range="0.3"
+                        max_range="1.5"
+                        field_of_view="50"
+                        ray_count="2" />
+    <!-- Sonar Plugin -->
   </xacro:macro>
 </robot>

File: wamv_gazebo/urdf/components/sonar_sensor.xacro (robot description, xacro)
@@ -1,12 +1,17 @@
-<?xml version="1.0"?>
+<?xml version="1.0" encoding="UTF-8"?>
 <robot xmlns:xacro="http://ros.org/wiki/xacro">
-  <xacro:macro name="sonar" params="name x y z R:=0 P:=0 Y:=0 ros_topic update_rate min_range max_range field_of_view ray_count">
-    <joint name="${name}_joint" type="fixed">
+  <xacro:macro name="sonar" params="name x:=0 y:=0 z:=0 R:=0 P:=0 Y:=0 ros_topic update_rate:=10 min_range:=0.3 max_range:=2 field_of_view:=56 ray_count:=2">
+    <joint name="${namespace}/${name}_joint" type="fixed">
       <origin xyz= "${x} ${y} ${z}" rpy="${R} ${P} ${Y}" />
-      <parent link="base_link"/>
-      <child link="${name}_link"/>
+      <parent link="${namespace}/base_link"/>
+      <child link="${namespace}/${name}_link"/>
     </joint>
-    <link name="${name}_link">
+    <link name="${namespace}/${name}_link">
       <inertial>
+          <visual name="${namespace}/${name}_visual">
+        <geometry>
+          <mesh filename="package://wamv_gazebo/models/sonar/mesh/sonar.dae"/>
+        </geometry>
+      </visual>
         <mass value="0.001" />
         <origin xyz="0 0 0" rpy="0 0 0" />
@@ -20,5 +25,5 @@
       </visual>
       <visual>
-        <origin xyz="0.05 0 0" rpy="0 1.57 ${Y}" />
+        <origin xyz="0 0 0" rpy="0 0 0" />
         <geometry>
           <cylinder length="0.06" radius="0.02" />
@@ -32,10 +37,10 @@
       </collision>
     </link>
-    <gazebo reference="${name}_link">
+    <gazebo reference="${namespace}/${name}_link">
       <sensor type="ray" name="${name}">
         <always_on>true</always_on>
         <update_rate>${update_rate}</update_rate>
         <pose>0 0 0 0 0 0</pose>
-        <visualize>false</visualize>
+        <visualize>true</visualize>
         <ray>
           <scan>
@@ -62,8 +67,11 @@
           <gaussianNoise>0.005</gaussianNoise>
           <topicName>${ros_topic}</topicName>
-          <frameId>${name}_link</frameId>
+          <frameId>${namespace}/${name}_link</frameId>
         </plugin>
       </sensor>
     </gazebo>
+    <gazebo reference="${namespace}/${name}_link">
+      <material>Gazebo/Black</material>
+    </gazebo>
   </xacro:macro>
 </robot>

File: wamv_gazebo/urdf/dynamics/wamv_gazebo_dynamics_plugin.xacro (robot description, xacro)
@@ -1,5 +1,5 @@
 <?xml version="1.0"?>
 <robot xmlns:xacro="http://ros.org/wiki/xacro">
-  <xacro:macro name="usv_dynamics_gazebo" params="name width:=2.4 length:=4.9">
+  <xacro:macro name="usv_dynamics_gazebo" params="name width:=1.1 length:=1.5">
     <!--Gazebo Plugin for simulating WAM-V dynamics-->
     <gazebo>
@@ -14,16 +14,16 @@
         <nDotR>0.0</nDotR>
         <!-- Linear and quadratic drag -->
-        <xU>51.3</xU>
-        <xUU>72.4</xUU>
-        <yV>40.0</yV>
+        <xU>9.74</xU>
+        <xUU>13.75</xUU>
+        <yV>7.6</yV>
         <yVV>0.0</yVV>
-        <zW>500.0</zW>
-        <kP>50.0</kP>
-        <mQ>50.0</mQ>
-        <nR>400.0</nR>
+        <zW>95</zW>
+        <kP>9.5</kP>
+        <mQ>9.5</mQ>
+        <nR>76</nR>
         <nRR>0.0</nRR>
         <!-- General dimensions -->
         <!--<boatArea>2.2</boatArea>-->
-        <hullRadius>0.213</hullRadius>
+        <hullRadius>0.08</hullRadius>
         <boatWidth>${width}</boatWidth>
         <boatLength>${length}</boatLength>

File: wamv_gazebo/urdf/thruster_layouts/wamv_t_thrusters.xacro (robot description, xacro)
@@ -4,5 +4,6 @@
   <xacro:engine prefix="left" position="${0.95+0.38} ${0.33} 0.368237" orientation="0.0 0.0 0.0" />
   <xacro:engine prefix="right" position="${0.95+0.38} ${-0.33} 0.368237"  orientation="0.0 0.0 0.0" />
-  <xacro:engine prefix="lateral" position="${0.68} ${0} 0.265237" orientation="0.0 0.0 0.0"/>
+  <xacro:engine prefix="middle" position="${0.68} ${0} 0.265237" orientation="0.0 0.0 0.0"/>
+  <xacro:engine prefix="lateral" position="${0.75} ${-0.25} 0.3" orientation="0.0 0.0 80.0"/>
   <gazebo>
     <plugin name="wamv_gazebo_thrust" filename="libusv_gazebo_thrust_plugin.so">
@@ -12,4 +13,5 @@
       <xacro:wamv_gazebo_thruster_config name="left" />
       <xacro:wamv_gazebo_thruster_config name="right" />
+      <xacro:wamv_gazebo_thruster_config name="middle" />
       <xacro:wamv_gazebo_thruster_config name="lateral" />
     </plugin>

File: wamv_gazebo/urdf/wamv_gazebo.urdf.xacro (robot description, xacro)
@@ -15,5 +15,5 @@
   <xacro:arg name="camera_namespace" default="cameras/"/>
   <xacro:arg name="sensor_namespace" default="sensors/"/>
-  <xacro:arg name="shooter_namespace" default="shooters/"/>
+  <xacro:arg name="pinger_namespace" default="pingers/"/>
   <!-- Note: this is only used for some sensors that do not correctly use the
   robotNamespace parameter -->
@@ -22,35 +22,13 @@
   <xacro:property name="camera_namespace" value="$(arg camera_namespace)" scope="global" />
   <xacro:property name="sensor_namespace" value="$(arg sensor_namespace)" scope="global" />
-  <xacro:property name="shooter_namespace" value="$(arg shooter_namespace)" scope="global" />
+  <xacro:property name="pinger_namespace" value="$(arg pinger_namespace)" scope="global" />
   <xacro:property name="namespace" value="$(arg namespace)" scope="global" />
   <!-- Sensor yaml file -->
-  <xacro:arg name="yaml_component_generation" default="false"/>
-  <xacro:arg name="component_xacro_file" default = ""/>
-  <!-- Thruster yaml file -->
-  <xacro:arg name="yaml_thruster_generation" default="false"/>
-  <xacro:arg name="thruster_xacro_file" default = ""/>
+  <xacro:arg name="yaml_sensor_generation" default="false"/>
+  <xacro:arg name="sensor_xacro_file" default = ""/>
   <!-- === The WAM-V platform === -->
   <xacro:include filename="$(find wamv_gazebo)/urdf/wamv_gazebo.xacro"/>
   <!-- === Thrusters === -->
-  <!-- Use thruster yaml file if given -->
-  <xacro:if value="$(arg yaml_thruster_generation)">
-    <xacro:wamv_gazebo thruster_layout="$(arg thruster_xacro_file)"/>
-  </xacro:if>
-  <!-- Otherwise, add thrusters based on thruster_config variable -->
-  <xacro:unless value="$(arg yaml_thruster_generation)">
-    <xacro:property name="thruster_conf" value="$(arg thruster_config)"/>
-    <!-- Default WAM-V with two aft thrusters -->
-    <xacro:if value="${thruster_conf == 'H'}">
-       <xacro:wamv_gazebo thruster_layout="$(find wamv_gazebo)/urdf/thruster_layouts/wamv_aft_thrusters.xacro"/>
-    </xacro:if>
-    <!-- WAMV with "T" thruster configuration -->
-    <xacro:if value="${thruster_conf == 'T'}">
-      <xacro:wamv_gazebo thruster_layout="$(find wamv_gazebo)/urdf/thruster_layouts/wamv_t_thrusters.xacro"/>
-    </xacro:if>
-    <!-- WAMV with "X" thruster configuration -->
-    <xacro:if value="${thruster_conf == 'X'}">
-      <xacro:wamv_gazebo thruster_layout="$(find wamv_gazebo)/urdf/thruster_layouts/wamv_x_thrusters.xacro"/>
-    </xacro:if>
-  </xacro:unless>
+  <xacro:wamv_gazebo thruster_layout="$(find wamv_gazebo)/urdf/thruster_layouts/wamv_t_thrusters.xacro"/>
   <!-- === Decide if we lock the robot to the world === -->
   <xacro:if value="$(arg locked)">
@@ -58,5 +36,5 @@
       <link name="wamv_external_link"/>
       <joint name="wamv_external_pivot_joint" type="universal">
-        <parent>wamv::wamv/base_link</parent>
+        <parent>wamv::base_link</parent>
         <child>wamv_external_link</child>
         <axis>
@@ -81,45 +59,35 @@
   </xacro:if>
   <!-- === Sensors === -->
-  <!-- Use sensor yaml file if given -->
-  <xacro:if value="$(arg yaml_component_generation)">
-    <xacro:include filename="$(arg component_xacro_file)"/>
-    <xacro:yaml_components />
-    <!-- sonar_enabled -->
-      <xacro:if value="$(arg sonar_enabled)">
-    <xacro:sonar name="sonar_sensor" x="1.6" y="0.4" z="1.6" ros_topic="/distance1" Y="${radians(0)}"  update_rate="10" min_range="0.3" max_range="2" field_of_view="56" ray_count="2" />
-    <xacro:sonar name="sonar_sensor2" x="1.6" y="-0.4" z="1.6" ros_topic="/distance2" Y="${radians(0)}" update_rate="10" min_range="0.3" max_range="2" field_of_view="56" ray_count="2" />
-    <xacro:sonar name="sonar_sensor3" x="0.3" y="0.4" z="1.6" ros_topic="/distance3" Y="${radians(180)}" update_rate="10" min_range="0.3" max_range="2" field_of_view="56" ray_count="2" />
-    <xacro:sonar name="sonar_sensor4" x="0.3" y="-0.4" z="1.6" ros_topic="/distance4" Y="${radians(180)}" update_rate="10" min_range="0.3" max_range="2" field_of_view="56" ray_count="2" />
+  <!-- === Sonar === -->
+  <xacro:if value="$(arg sonar_enabled)">
+	<xacro:sonar name="sonar_sensor1" x="1.6" y="0.4" z="0.6" ros_topic="sonar1/distance1" Y="${radians(45)}" update_rate="10" min_range="0.3" max_range="2" field_of_view="56" ray_count="2" />
+	<xacro:sonar name="sonar_sensor2" x="1.6" y="0" z="0.6" ros_topic="sonar2/distance2" Y="${radians(0)}" update_rate="10" min_range="0.3" max_range="2" field_of_view="56" ray_count="2" />
+    	<xacro:sonar name="sonar_sensor3" x="1.6" y="-0.4" z="0.6" ros_topic="sonar3/distance3" Y="${radians(-45)}" update_rate="10" min_range="0.3" max_range="2" field_of_view="56" ray_count="2" />
+	<xacro:sonar name="sonar_sensor4" x="0.9" y="-0.4" z="0.6" ros_topic="sonar4/distance4" Y="${radians(-90)}" update_rate="10" min_range="0.3" max_range="2" field_of_view="56" ray_count="2" />
+    	<xacro:sonar name="sonar_sensor5" x="0.3" y="0.4" z="0.6" ros_topic="sonar5/distance5" Y="${radians(135)}" update_rate="10" min_range="0.3" max_range="2" field_of_view="56" ray_count="2" />
+	<xacro:sonar name="sonar_sensor6" x="0.3" y="0" z="0.6" ros_topic="sonar6/distance6" Y="${radians(180)}" update_rate="10" min_range="0.3" max_range="2" field_of_view="56" ray_count="2" />
+    	<xacro:sonar name="sonar_sensor7" x="0.3" y="-0.4" z="0.6" ros_topic="sonar7/distance7" Y="${radians(-135)}" update_rate="10" min_range="0.3" max_range="2" field_of_view="56" ray_count="2" />
+	<xacro:sonar name="sonar_sensor8" x="0.9" y="0.4" z="0.6" ros_topic="sonar8/distance8" Y="${radians(90)}" update_rate="10" min_range="0.3" max_range="2" field_of_view="56" ray_count="2" />
   </xacro:if>
-    <!-- Add CPU Cases -->
-    <xacro:include filename="$(find wamv_description)/urdf/cpu_cases.xacro" />
-    <xacro:cpu_cases position="0.75 0 0.65" orientation="0 0 0"/>
-  </xacro:if>
-  <!-- Otherwise, add sensors based on enable variables -->
-  <xacro:unless value="$(arg yaml_component_generation)">
-    <!-- Add simulated GPS -->
-    <xacro:if value="$(arg gps_enabled)">
-      <xacro:wamv_gps name="gps_wamv" x="0.65" y="0" z="0.3" />
-    </xacro:if>
-    <!-- Add Simulated IMU -->
-    <xacro:if value="$(arg imu_enabled)">
-      <xacro:wamv_imu name="imu_wamv" x="1.2" y="0" z="0.3" />
-    </xacro:if>
-    <!-- Add 3D LIDAR -->
-    <xacro:if value="$(arg lidar_enabled)">
-      <xacro:lidar name="lidar_wamv" x="0.6" y="0" z="0.65" type="16_beam"/>
-    </xacro:if>
-      <!-- Add PLANAR -->
-  	<xacro:if value="$(arg planar_enabled)">
-    	<xacro:wamv_multibeam_laser name="planar_wamv" x="0.6" y="0" z="0.65"/>
-  	</xacro:if>
-    <!-- ==== VRX sensor configuration ==== -->
-    <xacro:if value="$(arg vrx_sensors_enabled)">
-      <!-- Add a camera facing right -->
-      <xacro:if value="$(arg camera_enabled)">
+  <!-- Cameras -->
+  <xacro:if value="$(arg camera_enabled)">
       <xacro:wamv_camera name="front_camera" y="0" x="1.6" z="0.65" />
       <xacro:wamv_camera name="back_camera" y="0" x="0.30" z="0.65" P="${radians(-180)}"/>
-    </xacro:if>
-    </xacro:if>
-  </xacro:unless>
+  </xacro:if>
+  <!--  GPS -->
+  <xacro:if value="$(arg gps_enabled)">
+    <xacro:wamv_gps name="gps_wamv" x="0.65" y="0" z="0.3" />
+  </xacro:if>
+  <!--  IMU -->
+  <xacro:if value="$(arg imu_enabled)">
+    <xacro:wamv_imu name="imu_wamv" x="1.2" y="0" z="0.3" />
+  </xacro:if>
+  <!--  3D LIDAR -->
+  <xacro:if value="$(arg lidar_enabled)">
+    <xacro:lidar name="lidar_wamv" x="0.6" y="0" z="0.65" type="16_beam"/>
+  </xacro:if>
+  <!--  PLANAR -->
+  <xacro:if value="$(arg planar_enabled)">
+    <xacro:wamv_multibeam_laser name="planar_wamv" x="0.6" y="0" z="0.65"/>
+  </xacro:if>
 </robot>
